File: photogate.kicad_pcb (KiCad board)
At the start: 2 copper layers, 85 x 69 mm, 9 parts, among them J1 Conn_01x03_Pin

Commit message: V1 final touches
Parts:
- removed D2: IR26-21C_L110_TR8, LED_THT:LED_D5.0mm_Horizontal_O3.81mm_Z3.0mm
- removed H3, H4: MountingHole, MountingHole:MountingHole_2.2mm_M2
- removed R3: LDR07, LED_THT:LED_D5.0mm_Horizontal_O3.81mm_Z3.0mm
- added D1: IR26-21C_L110_TR8, LED_THT:LED_D5.0mm_Horizontal_O3.81mm_Z3.0mm, F.Cu at (87.0, 56.2)
- added G***: LOGO, LOGO, F.Cu at (92.8, 75.2)
- added Q1: Q1, LED_THT:LED_D5.0mm_Horizontal_O3.81mm_Z3.0mm, F.Cu at (164.3, 53.7)
- MountingHole 1: renamed from H1; footprint MountingHole:MountingHole_2.2mm_M2 -> MountingHole:MountingHole_5.5mm
- MountingHole 2: renamed from H2; footprint MountingHole:MountingHole_2.2mm_M2 -> MountingHole:MountingHole_5.5mm
- moved MountingHole 2 130.6 mm to (162.5, 111.5)
- moved MountingHole 1 29.8 mm to (88.5, 111.5)
Other:
- board text added: "GND"
- board text added: "SENSOR"
- board text added: "VCC +5V"
- board text added: "photogate V1.1"

Commit message: adding revision so kicad export script works
Parts:
- added kibuzzard-67ED3B28: G***, kibuzzard-67ED3B28, F.Cu at (159.8, 80.2)
Other:
- board text removed: "photogate V1.1"
